Commit message: fix: raise table height to 95mm and increase pick tolerance to 3mm
- Update table_z_m to 0.095m in vision pipeline and environment URDF
- Increase goal position tolerance to 3mm in pick_and_place_server
- Resolves reachability issue where elbow_joint exceeded upper limit

File: src/eezybotarm_description/urdf/environment.xacro (robot description, xacro)
@@ -26,12 +26,12 @@
       <origin xyz="0.210 0.0 -0.009" rpy="0 0 0"/>
     </joint>
-    <!-- Elevated Sorting Work Table (200 x 300 x 75 mm) -->
+    <!-- Elevated Sorting Work Table (200 x 300 x 95 mm) -->
     <!-- Front edge of board is at X = +0.460 m. Table is 110mm from front edge, depth is 200mm. -->
-    <!-- Table spans X in [+0.150, +0.350], center is at X = +0.250 m, Z top at +0.075 m (center at Z = 0.0375 m) -->
+    <!-- Table spans X in [+0.150, +0.350], center is at X = +0.250 m, Z top at +0.095 m (center at Z = 0.0475 m) -->
     <link name="work_table">
       <visual>
         <origin xyz="0 0 0" rpy="0 0 0"/>
         <geometry>
-          <box size="0.200 0.300 0.075"/>
+          <box size="0.200 0.300 0.095"/>
         </geometry>
         <material name="table_surface">
@@ -42,5 +42,5 @@
         <origin xyz="0 0 0" rpy="0 0 0"/>
         <geometry>
-          <box size="0.200 0.300 0.075"/>
+          <box size="0.200 0.300 0.095"/>
         </geometry>
       </collision>
@@ -49,5 +49,5 @@
       <parent link="${parent}"/>
       <child link="work_table"/>
-      <origin xyz="0.250 0.0 0.0375" rpy="0 0 0"/>
+      <origin xyz="0.250 0.0 0.0475" rpy="0 0 0"/>
     </joint>
     <!-- Camera Stand (height 300 mm, base width ~120 mm) -->

Commit message: feature(config): implemented SSOT and fixes for workspace gemetry

File: src/eezybotarm_description/urdf/environment.xacro (robot description, xacro)
@@ -2,6 +2,8 @@
 <robot xmlns:xacro="http://www.ros.org/wiki/xacro">
   <xacro:macro name="environment" params="parent:=base_link">
+    <xacro:property name="env_file" value="$(find eezybotarm_description)/config/environment.yaml" />
+    <xacro:property name="env" value="${xacro.load_yaml(env_file)['/**']['ros__parameters']}" />
     <!-- Base Mounting Board (500 x 300 x 18 mm) -->
-    <!-- Base link is 40mm from the rear edge along +X. Center is at X = -0.040 + 0.250 = +0.210 m -->
+    <!-- Waist joint center is 63mm from the rear edge. Center X = -0.063 + 0.250 = +0.187 m -->
     <link name="base_board">
       <visual>
@@ -24,14 +26,12 @@
       <parent link="${parent}"/>
       <child link="base_board"/>
-      <origin xyz="0.210 0.0 -0.009" rpy="0 0 0"/>
+      <origin xyz="0.187 0.0 -0.009" rpy="0 0 0"/>
     </joint>
-    <!-- Elevated Sorting Work Table (200 x 300 x 95 mm) -->
-    <!-- Front edge of board is at X = +0.460 m. Table is 110mm from front edge, depth is 200mm. -->
-    <!-- Table spans X in [+0.150, +0.350], center is at X = +0.250 m, Z top at +0.095 m (center at Z = 0.0475 m) -->
+    <!-- Work Table / Workspace (depth along X, width along Y, height along Z) -->
     <link name="work_table">
       <visual>
         <origin xyz="0 0 0" rpy="0 0 0"/>
         <geometry>
-          <box size="0.200 0.300 0.095"/>
+          <box size="${env['table_depth_m']} ${env['table_width_m']} ${env['table_z_m']}"/>
         </geometry>
         <material name="table_surface">
@@ -42,5 +42,5 @@
         <origin xyz="0 0 0" rpy="0 0 0"/>
         <geometry>
-          <box size="0.200 0.300 0.095"/>
+          <box size="${env['table_depth_m']} ${env['table_width_m']} ${env['table_z_m']}"/>
         </geometry>
       </collision>
@@ -49,7 +49,7 @@
       <parent link="${parent}"/>
       <child link="work_table"/>
-      <origin xyz="0.250 0.0 0.0475" rpy="0 0 0"/>
+      <origin xyz="${env['robot_x_offset_m'] + env['table_depth_m']/2.0} ${env.get('robot_y_offset_m', 0.0)} ${env['table_z_m']/2.0}" rpy="0 0 0"/>
     </joint>
-    <!-- Camera Stand (height 300 mm, base width ~120 mm) -->
+    <!-- Camera Stand (height 300 mm, triangular base width 125 mm along front edge) -->
     <!-- Located at X = +0.400 m, Y = 0.0, Z center at +0.150 m -->
     <link name="camera_stand">
@@ -57,5 +57,5 @@
         <origin xyz="0 0 0" rpy="0 0 0"/>
         <geometry>
-          <cylinder radius="0.060" length="0.300"/>
+          <cylinder radius="0.0625" length="0.300"/>
         </geometry>
         <material name="stand_green">
@@ -66,5 +66,5 @@
         <origin xyz="0 0 0" rpy="0 0 0"/>
         <geometry>
-          <cylinder radius="0.060" length="0.300"/>
+          <cylinder radius="0.0625" length="0.300"/>
         </geometry>
       </collision>

Commit message: fix: added missing package descriptions

File: src/eezybotarm_description/urdf/environment.xacro (robot description, xacro)
@@ -97,5 +97,5 @@
       <parent link="camera_stand"/>
       <child link="camera_link"/>
-      <origin xyz="0.0 0.0 0.150" rpy="0.0 0.9828 3.14159"/>
+      <origin xyz="0.0 0.0 0.150" rpy="0.0 -0.9828 3.14159"/>
     </joint>
     <!-- Camera Optical Frame (ROS Standard: Z forward, X right, Y down) -->

Commit message: fix(workspace): update workspace geometry and robot offset parameters

File: src/eezybotarm_description/urdf/environment.xacro (robot description, xacro)
@@ -52,10 +52,10 @@
     </joint>
     <!-- Camera Stand (height 300 mm, triangular base width 125 mm along front edge) -->
-    <!-- Located at X = +0.400 m, Y = 0.0, Z center at +0.150 m -->
+    <!-- Located at X = +0.390 m, Y = 0.0, Z center at +0.150 m -->
     <link name="camera_stand">
       <visual>
         <origin xyz="0 0 0" rpy="0 0 0"/>
         <geometry>
-          <cylinder radius="0.0625" length="0.300"/>
+          <cylinder radius="0.05" length="0.300"/>
         </geometry>
         <material name="stand_green">
@@ -66,5 +66,5 @@
         <origin xyz="0 0 0" rpy="0 0 0"/>
         <geometry>
-          <cylinder radius="0.0625" length="0.300"/>
+          <cylinder radius="0.05" length="0.300"/>
         </geometry>
       </collision>
@@ -73,5 +73,5 @@
       <parent link="${parent}"/>
       <child link="camera_stand"/>
-      <origin xyz="0.400 0.0 0.150" rpy="0 0 0"/>
+      <origin xyz="0.390 0.0 0.150" rpy="0 0 0"/>
     </joint>
     <!-- Camera Body Link mounted on top of the stand (Z = +0.150 relative to stand center, i.e., Z = +0.300 m) -->
