Commit message: vision: add object detection and sorting pipeline with TensorRT acceleration

File: src/eezybotarm_description/urdf/robot.urdf (robot description, URDF)
Before this commit: robot eezybotarm, 10 links, 9 joints
Joints:
- joint elbow_joint: limit lower=0 upper=0.55 effort=0 velocity=0 -> lower=-0.2 upper=0.85 effort=0 velocity=0

File: src/eezybotarm_moveit_config/config/eezybotarm.urdf.xacro (robot description, xacro)
@@ -6,6 +6,12 @@
     <xacro:arg name="i2c_address" default="0x60" />
     <xacro:arg name="pwm_frequency" default="50" />
+    <xacro:arg name="include_environment" default="true" />
     <!-- Import eezybotarm urdf file -->
     <xacro:include filename="$(find eezybotarm_description)/urdf/robot.urdf" />
+    <!-- Import workspace environment xacro -->
+    <xacro:include filename="$(find eezybotarm_description)/urdf/environment.xacro" />
+    <xacro:if value="$(arg include_environment)">
+        <xacro:environment parent="base_link" />
+    </xacro:if>
     <!-- Import control_xacro -->
     <xacro:include filename="eezybotarm.ros2_control.xacro" />

Commit message: refactor(hw-interface): hardware interface and extract PCA9685 driver
- separate PCA9685 communication logic into a dedicated driver class and
clean up parameter parsing and error handling in the ros2_control hardware
interface.
- change controller update rate to 50 Hz to match servo control rate
- update joint limits and add standby group state

File: src/eezybotarm_description/urdf/robot.urdf (robot description, URDF)
Before this commit: robot eezybotarm, 10 links, 9 joints
Joints:
- joint elbow_joint: limit lower=-0.2 upper=0.85 effort=0 velocity=0 -> lower=-0.25 upper=0.85 effort=0 velocity=0
- joint waist_joint: limit lower=-0.7854 upper=0.7854 effort=0 velocity=0 -> lower=-1.2217 upper=1.2217 effort=0 velocity=0

File: src/eezybotarm_moveit_config/config/eezybotarm.ros2_control.xacro (robot description, xacro)
@@ -57,6 +57,6 @@
                 </state_interface>
                 <param name="pca_channel">3</param>
-                <param name="rad_min">-0.1500</param>
-                <param name="rad_max">0.6500</param>
+                <param name="rad_min">-1.5708</param>
+                <param name="rad_max">1.5708</param>
                 <param name="us_min">600</param>
                 <param name="us_max">2400</param>

Commit message: fix(urdf): fixed joint limits

File: src/eezybotarm_description/urdf/robot.urdf (robot description, URDF)
Before this commit: robot eezybotarm, 10 links, 9 joints
Joints:
- joint elbow_joint: limit lower=-0.25 upper=0.85 effort=0 velocity=0 -> lower=-0.25 upper=0.9 effort=0 velocity=0

Commit message: fix(urdf): extend elbow_joint limit to [-0.25; 1.0] radians

File: src/eezybotarm_description/urdf/robot.urdf (robot description, URDF)
Before this commit: robot eezybotarm, 10 links, 9 joints
Joints:
- joint elbow_joint: limit lower=-0.25 upper=0.9 effort=0 velocity=0 -> lower=-0.25 upper=1.0 effort=0 velocity=0

Commit message: perf(moveit_config,description): optimize collisions, decouple rviz, and increase gripper speed
- decouple RViz and move_group from bringup.launch.py into standalone rviz.launch.py, keeping bringup purely headless for Jetson
- conditionally include rviz.launch.py in local.launch.py and clean up jetson.launch.py arguments
- add disable_collisions entries in eezybotarm.srdf for unreachable camera stand/link and table pairs
- delete unused 2.9 MB mesh EBAmk2_001_base.STL
- harmonize waist_joint limits ([-1.2, 1.2]) and set non-zero effort/velocity limits in robot.urdf
- explicitly declare shoulder_joint position limits in joint_limits.yaml
- increase gripper open/close speed by ~+30% across joint_limits.yaml, robot.urdf, and dashboard_node.py

File: src/eezybotarm_description/urdf/robot.urdf (robot description, URDF)
Before this commit: robot eezybotarm, 10 links, 9 joints
Joints:
- joint ee_joint: origin xyz=0.06 0 0 rpy=0 0 0 -> xyz=0.07 0 0 rpy=0 0 0
- joint elbow_joint: limit lower=-0.25 upper=1.0 effort=0 velocity=0 -> lower=-0.25 upper=1.0 effort=1.5 velocity=1.57
- joint finger_left_joint: limit lower=0 upper=0.65 effort=0 velocity=1.0 -> lower=0 upper=0.65 effort=1.5 velocity=1.3
- joint finger_right_joint: limit lower=0 upper=0.65 effort=0 velocity=1.0 -> lower=0 upper=0.65 effort=1.5 velocity=1.3
- joint shoulder_joint: limit lower=-0.45 upper=0.80 effort=0 velocity=0 -> lower=-0.45 upper=0.80 effort=1.5 velocity=1.57
- joint waist_joint: limit lower=-1.2217 upper=1.2217 effort=0 velocity=0 -> lower=-1.2 upper=1.2 effort=1.5 velocity=1.57
- joint wrist_joint: limit lower=-3.14159 upper=3.14159 effort=0 velocity=0 -> lower=-3.14159 upper=3.14159 effort=1.5 velocity=1.57

Commit message: fix: minor callibrations
- update end-effector offset
- update home position coordinates
- decrease delay between sorting actions
- decrease amount of confirmation frames

File: src/eezybotarm_description/urdf/robot.urdf (robot description, URDF)
Before this commit: robot eezybotarm, 10 links, 9 joints
Joints:
- joint ee_joint: origin xyz=0.07 0 0 rpy=0 0 0 -> xyz=0.075 0 0 rpy=0 0 0
